File: controller-main.sch (EAGLE design)
At the start: 9 parts

Commit message: Updated main board
Parts:
- removed G1: SL-160AA/PR, battery:SL-160AA/PR
- removed SV1: (no value), con-lstb:MA10-1
- removed SV2: (no value), con-lstb:MA06-1
- added OUT: (no value), con-lstb:MA08-1
- added R1, R2, R3, R4: 10k, rcl:R-EU_0204/5
- added R5: 1k, rcl:R-EU_0204/5
- added R6: 2k, rcl:R-EU_0204/5
- added TOP1: (no value), con-lstb:MA06-1
- added TOP2: (no value), con-lstb:MA10-1
- added U$1: LEVEL-SHIFTER-4CH, diy-modules:LEVEL-SHIFTER-4CH
Connections:
- removed net AN: MCU.(PCI19/INT1/OC2B)PD3, SV2.2
- removed net BD: MCU.(PCI20/XCK/T0)PD4, SV1.7
- removed net BL: MCU.(PCI22/AIN0OC0A)PD6, SV1.9
- removed net BR: MCU.(PCI21/T1/OC0B)PD5, SV1.8
- removed net BU: MCU.(PCI23/AIN1)PD7, SV1.10
- removed net MA: MCU.(PCI18/INT0)PD2, SV2.6
- removed net SELECT: MCU.(PCI12/ADC4/SDA)PC4, SV1.2
- removed net TURBO: MCU.(PCI13/ADC5/SCL)PC5, SV1.1
- new net 3.3V: R5.1, U$1.LV
- new net 4D_CS: MCU.PB6(XTAL1/TOSC1/PCI6), OUT.6
- new net 4D_PD: MCU.PB7(XTAL2/TOSC2/PCI7), OUT.5
- new net AGND1: LAX.2, R1.1
- new net AGND2: R2.1, RAX.2
- new net GND_LOW: RF_IC.GND@1, U$1.GND.1
- new net MOSI_LOW: RF_IC.SIN, U$1.LV3
- new net N$1: MCU.PC6(/RESET/PCI14), TOP2.10
- new net N$12: LAY.2, R3.1
- new net N$15: MCU.(PCI21/T1/OC0B)PD5, OUT.4
- new net N$16: R4.1, RAY.2
- new net N$2: MCU.(PCI20/XCK/T0)PD4, TOP2.1
- new net N$3: MCU.(PCI19/INT1/OC2B)PD3, TOP2.2
- new net N$4: MCU.(PCI16/RXD)PD0, TOP2.9
- new net N$5: MCU.(PCI17/TXD)PD1, TOP2.8
- new net N$6: MCU.(PCI18/INT0)PD2, TOP2.7
- new net RF_CS_LOW: RF_IC.CS, U$1.LV2
- new net RF_RES: MCU.(PCI0/ICP/CLKO)PB0, U$1.HV4
- new net RF_RES_LOW: RF_IC.RESET, U$1.LV4
- new net SCK_LOW: RF_IC.SCK, U$1.LV1
- net 5V: now also MCU.AREF, OUT.8, R5.2, U$1.HV; no longer G1.+, LAY.2, RF_IC.VDD@2
- net AGND: now also R1.2, R2.2, R3.2, R4.2; no longer LAX.2, RAX.2, RAY.2
- net GND: now also OUT.7, R6.1, TOP1.4, U$1.GND.2; no longer G1.-, RF_IC.GND, SV2.4
- net LAX: now also MCU.(PCI8/ADC0)PC0; no longer MCU.(PCI11/ADC3)PC3
- net LAY: now also MCU.(PCI9/ADC1)PC1; no longer MCU.(PCI10/ADC2)PC2
- net MISO: now also OUT.2
- net MOSI: now also OUT.3, U$1.HV3; no longer RF_IC.SIN
- net RAX: now also MCU.(PCI10/ADC2)PC2; no longer MCU.(PCI9/ADC1)PC1
- net RAY: now also MCU.(PCI11/ADC3)PC3; no longer MCU.(PCI8/ADC0)PC0
- net RF_CS: now also MCU.(PCI1/OC1A/OC1S)PB1, U$1.HV2; no longer MCU.(PCI2/SS/OC1B)PB2, RF_IC.CS
- net RF_INT: now also MCU.(PCI2/SS/OC1B)PB2; no longer MCU.(PCI1/OC1A/OC1S)PB1
- net SCK: now also OUT.1, U$1.HV1; no longer RF_IC.SCK
Other:
- note removed: "TODO: vdd to 3.3V"
- moved on the sheet: LAX, LAY, MCU, RAX, RAY, RF_IC
