File: controller-main.brd (EAGLE design)
At the start: 100 x 80 mm, 24 parts

Commit message: Changed pin connections on the main board
Parts:
- added R17, R18: 1k, resistor:M1206
- moved I/O 7.62 mm to (36.8, 74.9)
- moved MCU 7.62 mm to (68.6, 52.1)
- moved R3 7.62 mm to (82.5, 39.4)
- moved R4 7.62 mm to (82.5, 34.3)
- moved RAN 7.62 mm to (63.5, 14.0)
- moved TOP1 7.62 mm to (77.5, 66.0)
- moved RF_L 7.62 mm to (10.2, 34.3)
- moved RF_R 7.62 mm to (10.2, 57.1)
- moved LAN 7.62 mm to (29.2, 14.0)
- moved R1 7.62 mm to (55.9, 39.4)
- moved R10 7.62 mm to (34.3, 48.3)
- moved R11 7.62 mm to (26.7, 43.2)
- moved R12 7.62 mm to (34.3, 43.2)
- moved R13 7.62 mm to (26.7, 38.1)
- moved R14 7.62 mm to (34.3, 38.1)
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Connections:
- removed net AD: MCU.29, TOP1.6
- removed net AL: MCU.31, TOP1.4
- removed net AR: MCU.30, TOP1.5
- removed net AU: MCU.32, TOP1.3
- removed net TUR: MCU.2, TOP1.1
- new net BATP: MCU.25, R17.1, R18.2
- net 4D_INT: now also MCU.1; no longer MCU.11
- net 5V: now also R18.1
- net BD: now also MCU.30; no longer MCU.28
- net BL: now also MCU.27; no longer MCU.26
- net BR: now also MCU.28; no longer MCU.27
- net BU: now also MCU.26; no longer MCU.25
- net GND: now also R17.2
- net RF_INT: now also MCU.32; no longer MCU.12
- net SEL: now also MCU.31; no longer MCU.1
Routing:
- net BATP: track 0.00 -> 25.2 mm, vias 0 -> 2
- net 4D_INT: track 54.6 -> 36.0 mm, vias 0 -> 1
- net RF_INT: track 41.1 -> 58.7 mm, vias 0 -> 2
- net AD: track 15.4 -> 0.00 mm
- net AL: track 14.0 -> 0.00 mm
- net TUR: track 13.8 -> 0.00 mm
- net AR: track 13.5 -> 0.00 mm
- net AU: track 12.1 -> 0.00 mm
- net 5V: track 221.3 -> 230.0 mm
- net GND: track 409.4 -> 414.3 mm
- net SEL: track 12.9 -> 10.7 mm
- net BU: track 21.6 -> 22.7 mm
- net BD: track 17.3 -> 18.3 mm
- net BR: track 18.5 -> 19.3 mm
- net BL: track 20.2 -> 21.0 mm
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Other:
- board size 100 x 80 mm -> 91.1 x 80 mm

Commit message: only half done
Parts:
- removed R10, R12, R14, R16, R17, R18, R6, R8: 1k, resistor:M1206
- removed R11, R13, R15, R5, R7, R9: 2k, resistor:M1206
- removed TOP1: (no value), con-lstb:MA10-1W
- removed TOP2: (no value), con-lstb:MA08-1W
- added C1: (no value), resistor:C1206
- added IC1: REG1117, burr-brown:SOT223
- added SV1: (no value), con-lstb:MA03-1
- moved RF_L 33.9 mm to (33.2, 59.1)
- moved RF_R 31.1 mm to (33.2, 36.3)
- moved R3 29.4 mm to (55.0, 29.0), turned to 180 degrees
- moved R4 28.4 mm to (57.0, 22.0), turned to 90 degrees
- moved MCU 26.1 mm to (48.0, 36.0), turned to 180 degrees
- moved R1 21.7 mm to (38.0, 27.0)
- moved R2 21.7 mm to (38.0, 22.0)
- moved I/O 21.1 mm to (48.0, 57.0)
- moved RAN 9.41 mm to (70.4, 20.4)
- moved LAN 7.34 mm to (25.6, 20.4)
Connections:
- removed net 4D_INT: I/O.5, MCU.1
- removed net BATP: MCU.25, R17.1, R18.2
- removed net BL: MCU.27, TOP1.9
- removed net BR: MCU.28, TOP1.8
- removed net BU: MCU.26, TOP1.10
- removed net MISO_LOW: R13.2, R14.1, RF_R.1
- removed net RF_CS_LOW: R11.2, R12.1, RF_R.2
- removed net RF_INT_LOW: R5.2, R6.1, RF_L.4
- removed net RF_RES_LOW: R7.2, R8.1, RF_L.2
- removed net SCK_LOW: R15.2, R16.1, RF_L.6
- net 3.3V: now also IC1.2; no longer R10.1, R9.2
- net 4D_CS: now also I/O.5, MCU.12; no longer I/O.4, MCU.10
- net 4D_PD: now also MCU.11; no longer MCU.9
- net 5V: now also C1.1, IC1.3; no longer R10.2, R18.1
- net BD: now also MCU.9, SV1.3; no longer MCU.30, TOP1.7
- net GND: now also C1.2, IC1.1, SV1.1; no longer R11.1, R13.1, R15.1, R17.2, R5.1, R7.1, R9.1, TOP2.4
- net LAX: now also MCU.26; no longer MCU.22
- net LAY: now also MCU.25; no longer MCU.19
- net MISO: now also RF_R.1; no longer R14.2
- net RAX: now also MCU.28; no longer MCU.23
- net RAY: now also MCU.27; no longer MCU.24
- net RF_CS: now also RF_R.2; no longer R12.2
- net RF_INT: now also MCU.1, RF_L.4; no longer MCU.32, R6.2
- net RF_RES: now also RF_L.2; no longer R8.2
- net SCK: now also RF_L.6; no longer R16.2
- net SEL: now also MCU.10, SV1.2; no longer MCU.31, TOP1.2
Routing:
- net GND: track 414.3 -> 80.4 mm
- net 5V: track 230.0 -> 42.0 mm
- net LAX: track 161.4 -> 31.9 mm
- net MOSI: track 113.3 -> 19.2 mm, vias 1 -> 0
- net SCK_LOW: track 88.1 -> 0.00 mm
- net RAY: track 84.4 -> 0.00 mm
- net MISO: track 77.8 -> 0.00 mm
- net SCK: track 99.9 -> 27.4 mm, vias 1 -> 0
- net RF_RES_LOW: track 69.7 -> 0.00 mm
- net RAX: track 63.9 -> 0.00 mm, vias 1 -> 0
- net RF_CS_LOW: track 62.7 -> 0.00 mm
- net MISO_LOW: track 60.9 -> 0.00 mm
- net RF_INT: track 58.7 -> 0.00 mm, vias 2 -> 0
- net 4D_CS: track 54.0 -> 0.00 mm
- net RF_INT_LOW: track 49.1 -> 0.00 mm
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Other:
- board size 91.1 x 80 mm -> 191.4 x 80 mm

Commit message: finished the main board
Parts:
- added R5, R6, R7, R8, R9: (no value), resistor:M1206
- R1, R2, R3, R4: value 10k -> (none)
- moved IC1 58.6 mm to (34.0, 45.0)
- moved R3 34.5 mm to (25.0, 46.0)
- moved R4 28.6 mm to (40.0, 45.0), turned to 0 degrees
- moved R2 26.0 mm to (62.0, 32.0), turned to 90 degrees
- moved R1 18.3 mm to (56.0, 23.8), turned to 270 degrees
- turned C1 to 90 degrees
Connections:
- new net 5V2: R2.2, R6.2, RAN.VCCX
- new net 5V_R: R2.1, RAN.VCCY
- new net GND_R: LAN.GNDX, LAN.GNDY, R1.2, RAN.GNDX, RAN.GNDY
- new net MISO2: I/O.6, R3.2
- new net MISO3: MCU.16, R4.2
- new net N$1: R1.1, R5.2
- new net N$2: LAN.OUTX, R9.1
- new net RST: MCU.29, R7.2
- new net RST2: R7.1, R8.2
- new net RST3: I/O.4, R8.1
- net 5V: now also R6.1; no longer RAN.VCCX, RAN.VCCY
- net GND: now also R5.1; no longer LAN.GNDX, LAN.GNDY, R1.1, R2.1, R3.1, R4.1, RAN.GNDX, RAN.GNDY
- net LAX: now also R9.2; no longer LAN.OUTX, R2.2
- net LAY: no longer R1.2
- net MISO: now also R3.1, R4.1; no longer I/O.6, MCU.16
- net RAX: no longer R3.2
- net RAY: no longer R4.2
- net RF_CS: now also MCU.23; no longer MCU.14
- net RF_RES: now also MCU.24; no longer MCU.13
Routing:
- net 5V: track 42.0 -> 129.8 mm
- net GND_R: track 0.00 -> 72.6 mm
- net RF_INT: track 0.00 -> 52.7 mm, vias 0 -> 1
- net 5V2: track 0.00 -> 52.1 mm
- net RF_RES: track 14.4 -> 60.0 mm
- net RAX: track 0.00 -> 43.7 mm
- net GND: track 80.4 -> 123.8 mm
- net MISO2: track 0.00 -> 40.4 mm
- net RST3: track 0.00 -> 36.2 mm
- net SCK: track 27.4 -> 54.4 mm
- net MISO: track 0.00 -> 22.5 mm
- net N$2: track 0.00 -> 20.6 mm
- net LAX: track 31.9 -> 13.0 mm
- net RAY: track 0.00 -> 18.9 mm
- net MOSI: track 19.2 -> 35.4 mm
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